File: Zhonx_III_platine/Zhonx_Platine.sch (KiCad schematic (older format))
At the start: 35 parts, among them SW3 ON/OFF, SW4 PUSH, U1 MCP1700, U2 PCF8574R, U3 OLED_128X64, U4 MCMT5-F-V

Commit message: Add ZHONX_III V2
Other:
- note added: "I2C"
- note removed: "3 wire SPI"
Changed lines of the file:
@@
 LIBS:contrib
 LIBS:valves
-LIBS:Librairies_Zhonx
 LIBS:Zhonx_Platine-cache
 EELAYER 25 0
@@
 $EndComp
 Text Notes 7800 1250 0    31   ~ 0
-3 wire SPI
+I2C
 Text GLabel 4300 3500 0    50   Output ~ 0
 NSRST
