File: Zhonx_III_mere/Zhonx_III.sch (KiCad schematic (older format))
At the start: 140 parts, among them K1 L_Motor, K2 R_Motor, K3 USART, P1 JTAG, Q1 FDV301N, Q2 FDV301N, U1 MCP73213, U10 BSL214N, U11 BSL214N, U12 24LC64T, U13 INA138, U14 STM32F405RGT6, U16 Line_1, U17 Line_2, U18 Line_3, U19 Line_4, U2 A3918_L, U20 Line_5, U3 A3918_R, U4 LTC2955CTS8-2, U5 SIB911DK, U6 SI1551DL, U7 LM2940, U8 MCP1700, U9 MCP1700, X1 QUARTZ_8Z

Commit message: modification affectations E/S STM32
Parts:
- L2: value 10uH -> BEAD
- R40, R41, R42, R43: value 4,7K -> 2,2K
Connections:
- net +3.3V: no longer U13.5 (V+)
- net +3.3VADC: now also U13.5 (V+)
- net Enable_IR_Line: now also U14.28 (PB2)
- net I_BAT: now also U14.20 (PA4/ADC1_IN4); no longer U14.16 (PA2/ADC3_IN2)
- net Line_IR_L1: now also U14.16 (PA2/ADC3_IN2); no longer U14.20 (PA4/ADC1_IN4)
- net NSRST: no longer P1.4
- net PW_LED: now also U14.2 (PC13/RTC_AF1); no longer U14.50 (PA15)
- net WP_EEPROM: now also U14.53 (PC12); no longer U14.55 (PB3/JTDO-SWO)
- net TEST_BAT renamed V_BAT
- new net PA13/JTMS-SWO: P1.4, U14.55 (PB3/JTDO-SWO)
- no-connect marks 14 -> 12
