File: Zhonx_III_mere/_autosave-Zhonx_III.kicad_pcb (KiCad board)
At the start: 2 copper layers, 133 parts, among them K1 L_Motor, K2 R_Motor, K3 USART, P1 JTAG, Q1 FDV301N, Q2 FDV301N, U1 MCP73213, U10 BSL214N, U11 BSL214N, U12 24LC64T, U14 STM32F405RGT6, U16 Line_1, U17 Line_2, U18 Line_3, U19 Line_4, U2 A3918, U20 Line_5, U3 A3918, U4 LTC2955CTS8-2, U5 SIB911DK, U6 SI1551DL, U7 LM2940, U8 MCP1700, U9 MCP1700, X1 16MHz

Commit message: Update Base_V2 (CamBam DXF)
Parts:
- moved R20 129.2 mm to (136.0, 185.8), turned to 270 degrees
- moved U17 127.0 mm to (131.7, 186.1), turned to 9 degrees
- moved C17 126.9 mm to (122.2, 188.2), turned to 180 degrees
- moved U16 124.9 mm to (144.2, 179.6), turned to 25 degrees
- moved C22 124.4 mm to (122.2, 186.9), turned to 180 degrees
- moved U18 124.4 mm to (122.2, 186.9), turned to 0 degrees
- moved IR2 124.1 mm to (134.4, 183.7), turned to 240 degrees
- moved R58 122.2 mm to (139.5, 180.6), turned to 180 degrees
- moved U19 121.6 mm to (112.7, 186.1), turned to 351 degrees
- moved R21 119.3 mm to (122.1, 184.3), turned to 0 degrees
- moved R64 118.8 mm to (108.6, 184.5), turned to 180 degrees
- moved C32 118.3 mm to (106.2, 184.0), turned to 90 degrees
- moved C31 118.1 mm to (107.2, 184.0), turned to 90 degrees
- moved IR3 117.0 mm to (109.9, 183.7), turned to 120 degrees
- moved U20 113.3 mm to (101.2, 180.6), turned to 335 degrees
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Other:
- board outline added: 70 x 97 mm
