File: Zhonx_III_base_V2/Zhonx_III_Base.sch (KiCad schematic (older format))
At the start: 50 parts, among them P100 CONN_BASE, P101 CONN_01X03, U101 MAX1607, U102 LT1370, U103 LP2992, U104 STM32F102C8, X101 8MHz

Commit message: Add ZHONX_III V2
Parts:
- D101, D103, D104: footprint LEDs:LED-0805 -> ZHONX:LED_HMSx-C120
Other:
- note added: "HSMR-C120"
Changed lines of the file:
@@
 F 0 "D101" H 2400 1950 50  0000 C CNN
 F 1 "LED" H 2400 1750 50  0000 C CNN
-F 2 "LEDs:LED-0805" H 2400 1850 60  0001 C CNN
+F 2 "ZHONX:LED_HMSx-C120" H 2400 1850 60  0001 C CNN
 F 3 "~" H 2400 1850 60  0000 C CNN
 	1    2400 1850
@@
 F 0 "D103" H 5650 4450 50  0000 C CNN
 F 1 "LED" H 5650 4250 50  0000 C CNN
-F 2 "LEDs:LED-0805" H 5650 4350 60  0001 C CNN
+F 2 "ZHONX:LED_HMSx-C120" H 5650 4350 60  0001 C CNN
 F 3 "~" H 5650 4350 60  0000 C CNN
 	1    5650 4350
@@
 F 0 "D104" H 5650 5000 50  0000 C CNN
 F 1 "LED" H 5650 4800 50  0000 C CNN
-F 2 "LEDs:LED-0805" H 5650 4900 60  0001 C CNN
+F 2 "ZHONX:LED_HMSx-C120" H 5650 4900 60  0001 C CNN
 F 3 "~" H 5650 4900 60  0000 C CNN
 	1    5650 4900
@@
 	-1   0    0    1
 $EndComp
+Text Notes 5000 4700 0    60   ~ 0
+HSMR-C120
 $EndSCHEMATC
