File: Zhonx_III_base_V2/Zhonx_III_Base.kicad_pcb (KiCad board)
At the start: 2 copper layers, 40 x 28 mm, 50 parts, among them P100 CONN_BASE, P101 CONN_01X03, U101 MAX1607, U102 LT1370, U103 LP2992, U104 STM32F102C8, X101 8MHz

Commit message: Create Zhonx mere V2
Other:
- copper layers 2 -> 4

Commit message: Update Base V2
Parts:
- P100: footprint ZHONX:CONN_BASE -> CONN_BASE
- USB101: footprint USB_MINI_AB -> ZHONX:USB_MINI_AB
- moved R104 3.26 mm to (103.0, 145.0)
- moved R105 3.26 mm to (106.0, 145.0)
- moved R103 1.50 mm to (107.5, 145.0)
- moved R106 1.50 mm to (104.5, 145.0)
- moved C101 1.22 mm to (100.1, 151.7)
- moved R101 0.86 mm to (115.0, 133.8)
- moved USB101 0.20 mm to (104.5, 150.2)
Routing:
- net +9V: track 39.9 -> 60.2 mm, vias 1 -> 2
- net +3.3V: track 67.7 -> 77.9 mm, vias 2 -> 7
- net Net-(R103-Pad1): track 10.6 -> 19.0 mm
- net +5V: track 32.2 -> 37.2 mm, vias 1 -> 3
- net Net-(R105-Pad1): track 3.00 -> 7.84 mm
- net Net-(R104-Pad2): track 3.00 -> 7.84 mm
- net USB_DM: track 16.9 -> 13.4 mm
- net STLINK_DAT: track 9.43 -> 7.18 mm
- net GND: track 193.4 -> 195.5 mm, vias 3 -> 11
- net Net-(C102-Pad1): track 50.9 -> 49.6 mm, vias 1 -> 4
- net Net-(P100-Pad2): track 17.1 -> 16.0 mm
- net Net-(D101-Pad2): track 17.0 -> 17.8 mm
- net Net-(P100-Pad4): track 38.0 -> 37.1 mm
- net Net-(C115-Pad1): track 9.24 -> 8.48 mm
- net Net-(C113-Pad1): track 2.90 -> 2.30 mm
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- added copper zone on B.Cu, net GND
- added copper zone on F.Cu, net GND
- added copper zone on GND.Cu, net GND
- added copper zone on VCC.Cu, net GND
Other:
- net class Default: via_dia 0.5 -> 0.6; via_drill 0.2 -> 0.3

Commit message: Add ZHONX_III V2
Parts:
- D101, D103, D104: footprint LEDs:LED-0805 -> ZHONX:LED_HMSx-C120
- P100: footprint CONN_BASE -> ZHONX:CONN_BASE
- R112, R113: moved to F.Cu
- R114, R115: moved to B.Cu
- USB101: value USB-MICRO_AB -> USB-MINI_AB
- moved R114 24.5 mm to (119.8, 155.5), turned to 180 degrees
- moved R115 23.1 mm to (119.8, 153.8)
- moved C107 15.9 mm to (95.0, 152.5)
- moved C102 12.1 mm to (87.0, 137.7), turned to 270 degrees
- moved R112 7.65 mm to (119.6, 147.9), turned to 270 degrees
- moved R113 5.85 mm to (121.3, 147.9), turned to 90 degrees
- moved D102 5.46 mm to (88.5, 152.5)
- moved C106 5.10 mm to (95.0, 145.5)
- moved C105 4.39 mm to (95.0, 149.0)
- moved C116 3.90 mm to (116.0, 149.9), turned to 180 degrees
- moved R103 3.67 mm to (103.9, 145.7)
- moved C115 3.61 mm to (113.2, 149.9), turned to 180 degrees
- moved R101 2.91 mm to (115.2, 130.9)
- moved R102 2.56 mm to (94.5, 153.8)
- moved X101 1.43 mm to (114.9, 152.2)
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Routing:
- net Net-(D103-Pad2): track 25.5 -> 1.26 mm, vias 1 -> 0
- net Net-(D104-Pad1): track 26.1 -> 7.34 mm, vias 1 -> 0
- net Net-(R114-Pad1): track 7.45 -> 22.0 mm, vias 0 -> 1
- net Net-(R103-Pad1): track 19.0 -> 5.76 mm
- net Net-(C102-Pad1): track 49.6 -> 42.8 mm
- net Net-(R112-Pad1): track 11.6 -> 5.09 mm, vias 1 -> 0
- net Net-(P100-Pad4): track 37.1 -> 31.4 mm
- net Net-(D102-Pad1): track 12.6 -> 17.9 mm
- net +5V: track 37.2 -> 42.4 mm
- net Net-(D101-Pad2): track 17.8 -> 21.4 mm
- net Net-(R105-Pad1): track 7.84 -> 4.61 mm
- net Net-(R104-Pad2): track 7.84 -> 4.65 mm
- net +9V: track 60.2 -> 57.3 mm, vias 2 -> 3
- net SWD_SWO: track 2.70 -> 5.52 mm
- net +3.3V: track 77.9 -> 75.5 mm
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Other:
- board size 40 x 28 mm -> 48 x 32 mm
- net class USB added: clearance 0.125, trace_width 0.3, via_dia 0.6, via_drill 0.3
- board text added: "ZHONX III BASE"

Commit message: Update Base_V2 (CamBam DXF)
Parts:
- moved R114 29.7 mm to (119.2, 125.8), turned to 270 degrees
- moved C103 29.3 mm to (94.5, 158.9), turned to 180 degrees
- moved R110 29.0 mm to (97.5, 160.2), turned to 0 degrees
- moved D102 28.1 mm to (116.2, 157.2), turned to 90 degrees
- moved R115 28.0 mm to (117.5, 125.8), turned to 270 degrees
- moved R111 28.0 mm to (99.8, 160.2), turned to 0 degrees
- moved C117 27.6 mm to (111.2, 122.5), turned to 0 degrees
- moved C104 27.5 mm to (93.7, 156.9), turned to 270 degrees
- moved D103 26.9 mm to (119.2, 128.7), turned to 90 degrees
- moved R119 26.6 mm to (108.7, 122.5), turned to 180 degrees
- moved R109 26.3 mm to (95.2, 156.9), turned to 270 degrees
- moved D101 26.0 mm to (119.2, 152.2), turned to 90 degrees
- moved R113 25.5 mm to (111.7, 124.3), turned to 180 degrees
- moved C102 25.5 mm to (101.5, 158.7), turned to 0 degrees
- moved C109 25.1 mm to (102.7, 123.3), turned to 0 degrees
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Other:
- board size 48 x 32 mm -> 32 x 48 mm
