File: Zhonx_III_mere_V2/Zhonx_III.sch (KiCad schematic (older format))
At the start: 155 parts, among them K1 L_Motor, K2 R_Motor, K3 USART, P1 JTAG, Q1 FDV301N, Q2 FDV301N, U1 MCP73213, U10 BSL214N, U11 BSL214N, U12 24LC64T, U13 INA138, U14 STM32F405RGT6, U16 Line_1, U17 Line_2, U18 Line_3, U19 Line_4, U2 A3918_L, U20 Line_5, U3 A3918_R, U4 LTC2955CTS8-1, U5 SIB911DK, U6 SI1551DL, U7 LM2940, U8 MCP1700, U9 MCP1700, X1 QUARTZ_8Z

Commit message: Add ZHONX_III V2
Parts:
- removed C100, C101: 100uF, symbol CP1
- removed C42: 10uF, symbol CP1
- removed C?: 10nF, symbol C
- removed C?: 10uF, symbol C
- removed C?: 100nF, symbol C
- removed Q1, Q2: FDV301N, ~, symbol MOSFET_N
- removed R12, R36: 100K, symbol R
- removed R15: 20K, symbol R
- removed R16: 10K, symbol R
- removed SCH1: BAT60, symbol DIODESCH
- removed U13: INA138, symbol INA138
- removed U5: SIB911DK, ~, symbol SIB911DK
- removed U6: SI1551DL, ~, symbol SI1551DL
- removed U7: LM2940, symbol LM2940
- removed U8, U9: MCP1700, symbol MCP1703
- removed U?: REG102, symbol REG102
- added C42: 2.2uF, Capacitors_SMD:C_0603, symbol C
- added C49, C50, C51: 0,47uF, Capacitors_SMD:C_0402, symbol C
- added C52, C53, C54: 10uF, Capacitors_SMD:C_0603, symbol C
- added Q1, Q2: BSS138, SMD_Packages:SOT-323, symbol Mosfet_N
- added U5: INA219, ZHONX:LTC2955, symbol INA219
- added U6: LT1761-5, Housings_SOT-23_SOT-143_TSOT-6:SOT-23-5, symbol LP2992
- added U7, U8: LT1761-3.3, Housings_SOT-23_SOT-143_TSOT-6:SOT-23-5, symbol LP2992
- ADXR1: footprint ~ -> ZHONX:ADXRS620
- C1, C20, C26, C27, C29, C9: footprint (none) -> Capacitors_SMD:C_0603
- C10, C11, C12, C13, C14, C21, C23, C24, C25, C28, C3, C35, C36, C37, C38, C39, C4, C40, C41, C43, C45, C5, C6, C7, C8: footprint (none) -> Capacitors_SMD:C_0402
- C103, C104: footprint (none) -> Capacitors_SMD:C_1206
- C15: value 0,1uF -> 10nF; footprint (none) -> Capacitors_SMD:C_0402
- C16: value 0,1uF -> 2,2uF; footprint (none) -> Capacitors_SMD:C_0603
- C17, C18, C2, C31: footprint ~ -> Capacitors_SMD:C_0603
- C19, C22, C30, C32, C33, C44: footprint ~ -> Capacitors_SMD:C_0402
- C34: value 1uF -> 2.2uF; footprint (none) -> Capacitors_SMD:C_0603
- C46: renamed from C?; value 2.2uF -> 2,2uF; footprint (none) -> Capacitors_SMD:C_0603
- C47, C48: renamed from C?; footprint (none) -> Capacitors_SMD:C_0402
- C55: renamed from C?; footprint (none) -> Capacitors_SMD:C_1206
- D1, L2, R27, R28: footprint ~ -> Resistors_SMD:R_0603
- D11: value Bleue_Charge -> BLUE; footprint (none) -> ZHONX:LED-0603-DVB
- D12: value Blanc_5V -> GREEN; footprint (none) -> ZHONX:LED-0603-DVB
- IR1: footprint (none) -> ZHONX:IR_LF
- IR2: footprint (none) -> ZHONX:IR_LD
- IR3: footprint (none) -> ZHONX:IR_RD
- IR4: footprint (none) -> ZHONX:IR_RF
- K1, K2: footprint (none) -> ZHONX:Connecteur_Moteur_Zhonx
- K3: footprint (none) -> ZHONX:Conn_Serial_Zhonx
- L1: renamed from L?; value 2,2uF -> 2,2uH; footprint ~ -> ZHONX:XFL4020
- P1: footprint (none) -> ZHONX:Zhonx_III_JTAG
- PL1: footprint ~ -> ZHONX:Platine_Zhonx_III
- R1: value 3,3K -> 620; footprint (none) -> Resistors_SMD:R_0402
- R10, R20, R21, R24, R25, R26, R30, R31, R32, R33, R8: footprint ~ -> Resistors_SMD:R_0402
- R11, R13, R14, R17, R18, R2, R23, R29, R40, R41, R42, R43, R44, R45, R48, R49, R50, R51, R52, R7, R9: footprint (none) -> Resistors_SMD:R_0402
- R12, R15, R16, R36: renamed from R?; footprint ~ -> Resistors_SMD:R_0402
- R19: value 820 -> 470; footprint (none) -> Resistors_SMD:R_0402
- R22: value 47K -> 1M; footprint (none) -> Resistors_SMD:R_0402
- R3: value 90K -> 90.9K 1%; footprint ~ -> Resistors_SMD:R_0402
- R34, R39: value 12 0,3W -> 10 1W; footprint (none) -> Resistors_SMD:R_0603
- R35: value 2,8 0,2W -> 2,2 2W; footprint (none) -> Resistors_SMD:R_0603
- R37: footprint (none) -> Resistors_SMD:R_1206
- R38: value 100 -> 0; footprint (none) -> Resistors_SMD:R_0402
- R4: value 1M -> 10; footprint ~ -> Resistors_SMD:R_0402
- R5: value 1M -> 6.2K; footprint ~ -> Resistors_SMD:R_0402
- R58, R67: value 220 -> 82; footprint (none) -> Resistors_SMD:R_0402
- R6: value 100K -> 10; footprint (none) -> Resistors_SMD:R_0402
- R64: value 33 -> 22; footprint (none) -> Resistors_SMD:R_0402
- SCH1: renamed from SCH?; footprint (none) -> ZHONX:PowerDI-123
- SP1: footprint ~ -> ZHONX:Buzzer_KSSG13J12
- U1: footprint (none) -> ZHONX:MCP73213
- U10, U11: footprint (none) -> Housings_SOT-23_SOT-143_TSOT-6:SOT-23-6
- U12: footprint (none) -> Housings_SOT-23_SOT-143_TSOT-6:SOT-23-5
- U14: footprint (none) -> ZHONX:TQFP_64
- U16, U17, U18, U19, U20: footprint (none) -> ZHONX:QRE1113GR
- U2, U3: footprint ~ -> ZHONX:QFN16_Termal_Pad
- U4: footprint (none) -> ZHONX:LTC2955
- U9: renamed from U?; footprint (none) -> ZHONX:DFN-10
- X1: footprint (none) -> ZHONX:Quartz_8Z-16MHz
Connections:
- net +3.3V: now also C51.2, C54.2, U8.5 (Vout); no longer C16.1
- net +3.3VADC: now also C10.1, C50.2, C53.2, U5.4 (Vs), U7.5 (Vout)
- net +5V: now also C34.2, C49.2, C52.2, U6.5 (Vout), U7.1 (Vin), U7.3 (ON/~OFF); no longer C15.1, C17.2, C18.1, C19.1, C2.1, C22.2, C30.1, C31.1, C32.1, C34.1, D1.2 (K), IR1.1 (A), IR3.1 (A), IR4.1 (A), K3.4 (P4), PL1.5 (4.5V), R19.2, R58.2, R64.2, R67.2, SP1.1
- net +8V: now also C16.1, C46.1, C9.2, R6.2, U1.3 (VBAT), U1.4 (VBAT), U4.6 (Vin), U9.4 (Vin), U6.1 (Vin); no longer C14.1, R5.1
- net +9V: now also U1.1 (VDD), U1.2 (VDD); no longer R6.1, U1.5 (NC)
- net +BATT: now also R37.2, R4.2; no longer C9.1, U1.10 (PROG)
- net EN_PW_ADC: now also R9.1, U6.3 (ON/~OFF)
- net Enable_IR_Line: now also Q1.1 (G)
- net GND: now also C10.2, C34.1, C9.1, R9.2, U1.9 (VSS), C42.1, C52.1, C53.1, C54.1, Q1.2 (S), Q2.2 (S), U5.3 (GND), U5.7 (A0), U5.8 (A1), U6.2 (GND), U7.2 (GND), U8.2 (GND); no longer C10.1, C14.2, C15.2, C34.2, C9.2, PL1.8 (WKUP), R4.1, R6.2
- net I2C_SCL: now also U5.5 (SCL)
- net I2C_SDA: now also U5.6 (SDA)
- net PIEZZO: now also C15.2; no longer R22.1, U11.3 (G2)
- net PW_LED: now also Q2.1 (G)
- net WKUP: now also PL1.8 (WKUP)
- net at D11.2 (K): now also U1.7 (STAT)
- net at R11.2: now also R5.2, U1.10 (PROG)
- net at U16.2 (K), U17.2 (K), U20.2 (K): now also Q1.3 (D)
- net FAST_CHARGE: now reaches U14.50 (PA15)
- net FAST_CHARGE: now also R5.1
- net at D12.2 (K): now also Q2.3 (D)
- net +4.5V: now reaches C55.2, L1.2, R16.2, U9.1 (BD), U9.7 (BIAS)
- net +4.5V: now also C17.2, C18.1, C19.1, C2.1, C22.2, C30.1, C31.1, C32.1, D1.2 (K), IR1.1 (A), IR3.1 (A), IR4.1 (A), K3.4 (P4), PL1.5 (4.5V), R19.2, R58.2, R64.2, R67.2, SP1.1, C42.2, U8.1 (Vin), U8.3 (ON/~OFF)
- net +5VA renamed +5VADC
- net GET_BAT_ADC: no longer names the net of U14.26 (PB0)
- net GET_BAT_ADC: no longer R4.2
- net I_BAT: no longer names the net of U14.20 (PA4/ADC1_IN4)
- net V_BAT: no longer names the net of U14.25 (PC5/ADC1_IN15)
- new net: C15.1, R22.1, U11.3 (G2)
- new net: C49.1, U6.4 (BYPASS)
- new net: C50.1, U7.4 (BYPASS)
- new net: C51.1, U8.4 (BYPASS)
- new net: C14.1, R4.1, U5.1 (Vin+)
- new net: C14.2, R6.1, U5.2 (Vin-)
- no-connect marks 13 -> 15
Other:
- note added: "10mA"
- note added: "150mA"
- note added: "2mA"
- note added: "330mA"
- note added: "Battery measurement"
- note added: "Charger"
- note added: "PANASONIC ERJ8BWFR100V 1206"
- note added: "Push Button Controller"
- note added: "Regulators"
- note added: "SOT-323"
- note added: "XFL4020-222"
- note removed: "Amperemeter"
- note removed: "Battery voltage measurement"
- note removed: "Power Managment"
- note removed: "Tantale - 1210"
- moved on the sheet: ADXR1, C1, C11, C20, C21, C23, C24, C25, C26, C27, C28, C29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

Commit message: Update Base_V2 (CamBam DXF)
Parts:
- C11: value 150nF -> 100nF
Changed lines of the file:
@@
 P 3000 3350
 F 0 "C11" H 3050 3450 50  0000 L CNN
-F 1 "150nF" H 3050 3250 50  0000 L CNN
+F 1 "100nF" H 3050 3250 50  0000 L CNN
 F 2 "Capacitors_SMD:C_0402" H 3000 3350 60  0001 C CNN
 F 3 "" H 3000 3350 60  0001 C CNN
